File: projects/benjolin/benjolin.kicad_pcb (KiCad board)
At the start: 2 copper layers, 87 parts, among them J1 LP OUT, J2 Conn_01x06, Q1 BC547, SW1 SPDT, U10 TL074, U11 TL072, U4 V2164, U5 TL074, U6 TL072, U7 TL072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

Commit message: add benjolin
Other:
- net class Default removed
