File: projects/benjolin/benjolin.kicad_sch (KiCad schematic)
At the start: 23 parts, among them J1 LP OUT, J3 PWM OUT

Commit message: it's a dual benjolin
Parts:
- removed J1: LP OUT, digikey-footprints:Test_Jack_Horiz, symbol dk_Banana-and-Tip-Connectors-Jacks-Plugs:105-1103-001
- removed J3: PWM OUT, digikey-footprints:Test_Jack_Horiz, symbol dk_Banana-and-Tip-Connectors-Jacks-Plugs:105-1103-001
- removed J?: XOR OUT, digikey-footprints:Test_Jack_Horiz, symbol dk_Banana-and-Tip-Connectors-Jacks-Plugs:105-1103-001
- removed J?: OSC1 FREQ IN 1, digikey-footprints:Test_Jack_Horiz, symbol dk_Banana-and-Tip-Connectors-Jacks-Plugs:105-1103-001
- removed J?: OSC1 FREQ IN 2, digikey-footprints:Test_Jack_Horiz, symbol dk_Banana-and-Tip-Connectors-Jacks-Plugs:105-1103-001
- removed J?: OSC2 FREQ IN 1, digikey-footprints:Test_Jack_Horiz, symbol dk_Banana-and-Tip-Connectors-Jacks-Plugs:105-1103-001
- removed J?: OSC2 FREQ IN 2, digikey-footprints:Test_Jack_Horiz, symbol dk_Banana-and-Tip-Connectors-Jacks-Plugs:105-1103-001
- removed R48, R50, R52, R53, R54, R55, R? (x4): 51k, 00-Mine:resistor-TH-10mm, symbol 00-cool_stuff:resistor
- removed RV10, RV12, RV14, RV15, RV16, RV17: 10k, 00-Mine:MOLEX-1X3_LOCK, symbol 00-cool_stuff:potentiometer
Other:
- removed sheet filter
- removed sheet oscillators
- removed sheet rungler
- added sheet benjolin-A (benjolin-core.kicad_sch)
- added sheet benjolin-B (benjolin-core.kicad_sch)
