File: projects/benjolin/rungler.kicad_sch (KiCad schematic)
At the start: 21 parts, among them Q1 BC547, SW1 SPDT, U7 TL072, U8 4021

Commit message: it's a dual benjolin
Connections:
- net Vcc: now also U7.8 (V+)
- net Vee: now also U7.4 (V-)
Changed lines of the file:
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@@
     (pin "2")
   )
-  (symbol (lib_id "00-cool_stuff:0V") (at 203.2 78.74 0)
+  (symbol (lib_id "00-cool_stuff:0V") (at 203.2 78.74 0) (unit 1)
     (in_bom yes) (on_board yes)
     (property "Reference" "#PWR032" (id 0) (at 203.2 85.09 0)
@@
     (pin "2")
     (pin "3")
+    (pin "5")
+    (pin "6")
+    (pin "7")
+    (pin "4")
+    (pin "8")
   )
   (symbol (lib_id "00-cool_stuff:TL072-separate") (at 213.36 74.93 0) (unit 2)
@@
       (effects (font (size 1.27 1.27)) hide)
     )
+    (pin "1")
+    (pin "2")
+    (pin "3")
     (pin "5")
     (pin "6")
     (pin "7")
+    (pin "4")
+    (pin "8")
   )
   (symbol (lib_id "00-cool_stuff:resistor") (at 96.52 50.8 0) (unit 1)
@@
     (pin "2")
   )
-  (symbol (lib_id "00-cool_stuff:0V") (at 86.36 91.44 0)
+  (symbol (lib_id "00-cool_stuff:0V") (at 86.36 91.44 0) (unit 1)
     (in_bom yes) (on_board yes)
     (property "Reference" "#PWR033" (id 0) (at 86.36 97.79 0)
@@
     (pin "3")
   )
-  (symbol (lib_id "00-cool_stuff:0V") (at 74.93 92.71 0)
+  (symbol (lib_id "00-cool_stuff:0V") (at 74.93 92.71 0) (unit 1)
     (in_bom yes) (on_board yes)
     (property "Reference" "#PWR034" (id 0) (at 74.93 99.06 0)
@@
     (pin "9")
   )
-  (symbol (lib_id "00-cool_stuff:Vcc") (at 212.09 114.3 0)
+  (symbol (lib_id "00-cool_stuff:Vcc") (at 212.09 114.3 0) (unit 1)
     (in_bom yes) (on_board yes)
     (property "Reference" "#PWR0116" (id 0) (at 212.09 118.11 0)
@@
     (pin "1")
   )
-  (symbol (lib_id "00-cool_stuff:Vee") (at 212.09 139.7 180)
+  (symbol (lib_id "00-cool_stuff:Vee") (at 212.09 139.7 180) (unit 1)
     (in_bom yes) (on_board yes)
     (property "Reference" "#PWR0117" (id 0) (at 212.09 142.24 0)
@@
     (pin "1")
   )
-  (symbol (lib_id "00-cool_stuff:TL072-separate") (at 214.63 125.73 0)
+  (symbol (lib_id "00-cool_stuff:TL072-separate") (at 214.63 125.73 0) (unit 3)
     (in_bom yes) (on_board yes)
     (property "Reference" "U7" (id 0) (at 220.472 124.5616 0)
@@
       (effects (font (size 1.27 1.27)) hide)
     )
+    (pin "1")
+    (pin "2")
+    (pin "3")
+    (pin "5")
+    (pin "6")
+    (pin "7")
     (pin "4")
     (pin "8")
   )
-  (symbol (lib_id "00-cool_stuff:cap_small") (at 219.71 116.84 0)
+  (symbol (lib_id "00-cool_stuff:cap_small") (at 219.71 116.84 0) (unit 1)
     (in_bom yes) (on_board yes)
     (property "Reference" "C21" (id 0) (at 219.71 111.0234 0))
@@
     (pin "2")
   )
-  (symbol (lib_id "00-cool_stuff:cap_small") (at 219.71 137.16 0)
+  (symbol (lib_id "00-cool_stuff:cap_small") (at 219.71 137.16 0) (unit 1)
     (in_bom yes) (on_board yes)
     (property "Reference" "C22" (id 0) (at 219.71 131.3434 0))
@@
     (pin "2")
   )
-  (symbol (lib_id "00-cool_stuff:0V") (at 229.87 139.7 0)
+  (symbol (lib_id "00-cool_stuff:0V") (at 229.87 139.7 0) (unit 1)
     (in_bom yes) (on_board yes)
     (property "Reference" "#PWR0118" (id 0) (at 229.87 146.05 0)
@@
     (pin "1")
   )
-  (symbol (lib_id "00-cool_stuff:0V") (at 229.87 119.38 0)
+  (symbol (lib_id "00-cool_stuff:0V") (at 229.87 119.38 0) (unit 1)
     (in_bom yes) (on_board yes)
     (property "Reference" "#PWR0119" (id 0) (at 229.87 125.73 0)
